File: hardware/rs232.kicad_pcb (KiCad board)
At the start: 2 copper layers, 45 x 35 mm, 37 parts, among them J1 DB9, P1 CON-SENSOR, P2 CONN_5, P3 CONN_5, P4 BOOT, P5 BOOT, U1 XMC1XXX48, U3 SP3232EBCN, U4 DRILL, U5 DRILL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

Commit message: specify processor
Parts:
- U1: value XMC1XXX48 -> XMC1404
Changed lines of the file:
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@@
   (module kicad-libraries:QFN48-EP2 (layer Vorderseite)
     (at 142.6 99.4)
-    (fp_text reference U1 (at 0 0) (layer F.SilkS)
-      (effects (font (size 0.29972 0.29972) (thickness 0.0762)))
+    (fp_text reference U1 (at 0 0) (layer F.Fab)
+      (effects (font (size 0.29972 0.29972) (thickness 0.07493)))
     )
-    (fp_text value XMC1XXX48 (at 0 -0.7) (layer F.SilkS)
-      (effects (font (size 0.29972 0.29972) (thickness 0.0762)))
+    (fp_text value XMC1404 (at 0 -0.7) (layer F.Fab)
+      (effects (font (size 0.29972 0.29972) (thickness 0.07493)))
     )
     (fp_circle (center -2.5 2.6) (end -2.4 2.8) (layer F.Fab) (width 0.05))
